Commit message: updated material name

File: urdf/youbot_gripper/gripper.urdf.xacro (robot description, xacro)
@@ -25,5 +25,5 @@
 					<mesh filename="package://youbot_description/meshes/youbot_gripper/palm.dae" />
 				</geometry>
-				<material name="Black" />
+				<material name="youBot/Black" />
 			</visual>
 			<collision>
@@ -55,5 +55,5 @@
 					<mesh filename="package://youbot_description/meshes/youbot_gripper/finger.dae" />
 				</geometry>
-				<material name="Black" />
+				<material name="youBot/Black" />
 			</visual>
 			<collision>
@@ -85,5 +85,5 @@
 					<mesh filename="package://youbot_description/meshes/youbot_gripper/finger.dae" />
 				</geometry>
-				<material name="Black" />
+				<material name="youBot/Black" />
 			</visual>
 			<collision>

File: urdf/youbot_plate/plate.urdf.xacro (robot description, xacro)
@@ -22,5 +22,5 @@
 					<mesh filename="package://youbot_description/meshes/youbot_plate/plate.dae" />
 				</geometry>
-				<material name="DarkGrey"/>
+				<material name="youBot/DarkGrey"/>
 			</visual>
 			<collision>
