Commit message: added dummy link

File: urdf/youbot_base/base.urdf.xacro (robot description, xacro)
@@ -32,4 +32,11 @@
   <xacro:property name="wheel_joint_safety_k_velocity" value="10.0"/>
   <xacro:macro name="youbot_base" params="name">
+    <link name="${name}_dummy">
+    </link>
+    <joint name="${name}_dummy_joint" type="fixed">
+      <origin xyz="0 0 0" rpy="0 0 0"/>
+      <child link="${name}_footprint"/>
+      <parent link="${name}_dummy"/>
+    </joint>
     <link name="${name}_footprint">
       <inertial>
